Commit message: Restore stable URDF (clean model working in Gazebo before ros2_control integration)

File: src/my_bot_description/urdf/my_bot.urdf.xacro (robot description, xacro)
@@ -10,5 +10,4 @@
   <xacro:property name="robot_mass" value="8.0"/> <!-- kg -->
   <!-- ========== Macros for inertial helpers ========== -->
-  <!-- Simple box inertia approximation -->
   <xacro:macro name="inertial_box" params="mass x y z">
     <inertial>
@@ -44,6 +43,5 @@
                         z="${base_height}"/>
   </link>
-  <!-- ========== Ball-handling "funnel" at the front ========== -->
-  <!-- Left guide -->
+  <!-- ========== Ball-handling "funnel" ========== -->
   <link name="funnel_left">
     <visual>
@@ -69,5 +67,4 @@
     <origin xyz="0 0 0" rpy="0 0 0"/>
   </joint>
-  <!-- Right guide -->
   <link name="funnel_right">
     <visual>
@@ -115,6 +112,5 @@
     <origin xyz="0 0 0" rpy="0 0 0"/>
   </joint>
-  <!-- ========== Wheels (left & right) ========== -->
-  <!-- Left wheel -->
+  <!-- ========== Wheels ========== -->
   <link name="left_wheel_link">
     <visual>
@@ -144,5 +140,4 @@
     <axis xyz="0 1 0"/>
   </joint>
-  <!-- Right wheel -->
   <link name="right_wheel_link">
     <visual>
@@ -170,5 +165,5 @@
     <axis xyz="0 1 0"/>
   </joint>
-  <!-- ========== Caster wheel (simple) ========== -->
+  <!-- Caster -->
   <link name="caster_wheel">
     <visual>
@@ -195,11 +190,10 @@
     <origin xyz="-${base_length/2.0 - 0.05} 0 0" rpy="0 0 0"/>
   </joint>
-     <!-- ========== Simple lidar link (for later SLAM) ========== -->
+  <!-- Simple lidar puck -->
   <link name="lidar_link">
     <visual>
-      <!-- Make it big and clearly above the base -->
-      <origin xyz="0 0 ${base_height + 0.30}" rpy="0 0 0"/>
-      <geometry>
-        <cylinder radius="0.15" length="0.30"/>
+      <origin xyz="0 0 ${base_height + 0.05}" rpy="0 0 0"/>
+      <geometry>
+        <cylinder radius="0.05" length="0.02"/>
       </geometry>
       <material name="lidar_body">
@@ -208,7 +202,7 @@
     </visual>
     <collision>
-      <origin xyz="0 0 ${base_height + 0.30}" rpy="0 0 0"/>
-      <geometry>
-        <cylinder radius="0.15" length="0.30"/>
+      <origin xyz="0 0 ${base_height + 0.05}" rpy="0 0 0"/>
+      <geometry>
+        <cylinder radius="0.05" length="0.02"/>
       </geometry>
     </collision>

Commit message: Final submission: robot, launch file, README

File: src/my_bot_description/urdf/my_bot.urdf.xacro (robot description, xacro)
@@ -1,221 +1,167 @@
 <?xml version="1.0"?>
 <robot xmlns:xacro="http://www.ros.org/wiki/xacro" name="my_bot">
-  <!-- ========= Global properties ========= -->
-  <xacro:property name="base_length" value="0.4"/>
-  <xacro:property name="base_width"  value="0.3"/>
-  <xacro:property name="base_height" value="0.15"/>
-  <xacro:property name="wheel_radius"      value="0.07"/>
-  <xacro:property name="wheel_width"       value="0.03"/>
-  <xacro:property name="wheel_separation"  value="0.28"/>
-  <xacro:property name="robot_mass" value="8.0"/> <!-- kg -->
-  <!-- ========== Macros for inertial helpers ========== -->
-  <xacro:macro name="inertial_box" params="mass x y z">
+  <!-- ================= GLOBAL ================= -->
+  <xacro:property name="base_length" value="0.55"/>
+  <xacro:property name="base_width"  value="0.40"/>
+  <xacro:property name="base_height" value="0.18"/>
+  <xacro:property name="wheel_radius" value="0.10"/>
+  <xacro:property name="wheel_width"  value="0.05"/>
+  <xacro:property name="wheel_sep"    value="0.36"/>
+  <xacro:property name="robot_mass" value="22.0"/>
+  <!-- ================= INERTIA MACRO ================= -->
+  <xacro:macro name="inertial_box" params="m x y z">
     <inertial>
-      <mass value="${mass}"/>
-      <origin xyz="0 0 0" rpy="0 0 0"/>
+      <mass value="${m}"/>
+      <origin xyz="0 0 0"/>
       <inertia
-        ixx="${mass * (y*y + z*z) / 12.0}"
-        iyy="${mass * (x*x + z*z) / 12.0}"
-        izz="${mass * (x*x + y*y) / 12.0}"
-        ixy="0.0" ixz="0.0" iyz="0.0"/>
+        ixx="${m*(y*y+z*z)/12}"
+        iyy="${m*(x*x+z*z)/12}"
+        izz="${m*(x*x+y*y)/12}"
+        ixy="0" ixz="0" iyz="0"/>
     </inertial>
   </xacro:macro>
-  <!-- ========== Base link (chassis) ========== -->
+  <!-- ================= BASE ================= -->
   <link name="base_link">
     <visual>
-      <origin xyz="0 0 ${base_height/2.0}" rpy="0 0 0"/>
+      <origin xyz="0 0 ${base_height/2}"/>
       <geometry>
         <box size="${base_length} ${base_width} ${base_height}"/>
       </geometry>
-      <material name="grey">
-        <color rgba="0.6 0.6 0.6 1.0"/>
-      </material>
     </visual>
     <collision>
-      <origin xyz="0 0 ${base_height/2.0}" rpy="0 0 0"/>
+      <origin xyz="0 0 ${base_height/2}"/>
       <geometry>
         <box size="${base_length} ${base_width} ${base_height}"/>
       </geometry>
     </collision>
-    <xacro:inertial_box mass="${robot_mass}"
+    <xacro:inertial_box m="${robot_mass}"
                         x="${base_length}"
                         y="${base_width}"
                         z="${base_height}"/>
   </link>
-  <!-- ========== Ball-handling "funnel" ========== -->
-  <link name="funnel_left">
+  <!-- ================= WHEELS ================= -->
+  <link name="left_wheel">
     <visual>
-      <origin xyz="${base_length/2.0} ${base_width/2.0} ${base_height}" rpy="0 0 0.6"/>
-      <geometry>
-        <box size="0.3 0.02 0.15"/>
-      </geometry>
-      <material name="blue">
-        <color rgba="0.2 0.3 0.8 1.0"/>
-      </material>
-    </visual>
-    <collision>
-      <origin xyz="${base_length/2.0} ${base_width/2.0} ${base_height}" rpy="0 0 0.6"/>
-      <geometry>
-        <box size="0.3 0.02 0.15"/>
-      </geometry>
-    </collision>
-    <xacro:inertial_box mass="0.5" x="0.3" y="0.02" z="0.15"/>
-  </link>
-  <joint name="funnel_left_joint" type="fixed">
-    <parent link="base_link"/>
-    <child link="funnel_left"/>
-    <origin xyz="0 0 0" rpy="0 0 0"/>
-  </joint>
-  <link name="funnel_right">
-    <visual>
-      <origin xyz="${base_length/2.0} ${-base_width/2.0} ${base_height}" rpy="0 0 -0.6"/>
-      <geometry>
-        <box size="0.3 0.02 0.15"/>
-      </geometry>
-      <material name="blue"/>
-    </visual>
-    <collision>
-      <origin xyz="${base_length/2.0} ${-base_width/2.0} ${base_height}" rpy="0 0 -0.6"/>
-      <geometry>
-        <box size="0.3 0.02 0.15"/>
-      </geometry>
-    </collision>
-    <xacro:inertial_box mass="0.5" x="0.3" y="0.02" z="0.15"/>
-  </link>
-  <joint name="funnel_right_joint" type="fixed">
-    <parent link="base_link"/>
-    <child link="funnel_right"/>
-    <origin xyz="0 0 0" rpy="0 0 0"/>
-  </joint>
-  <!-- Front bumper bar -->
-  <link name="front_bar">
-    <visual>
-      <origin xyz="${base_length/2.0 + 0.05} 0 ${base_height/2.0}" rpy="0 0 0"/>
-      <geometry>
-        <box size="0.05 ${base_width} 0.1"/>
-      </geometry>
-      <material name="black">
-        <color rgba="0.1 0.1 0.1 1.0"/>
-      </material>
-    </visual>
-    <collision>
-      <origin xyz="${base_length/2.0 + 0.05} 0 ${base_height/2.0}" rpy="0 0 0"/>
-      <geometry>
-        <box size="0.05 ${base_width} 0.1"/>
-      </geometry>
-    </collision>
-    <xacro:inertial_box mass="0.8" x="0.05" y="${base_width}" z="0.1"/>
-  </link>
-  <joint name="front_bar_joint" type="fixed">
-    <parent link="base_link"/>
-    <child link="front_bar"/>
-    <origin xyz="0 0 0" rpy="0 0 0"/>
-  </joint>
-  <!-- ========== Wheels ========== -->
-  <link name="left_wheel_link">
-    <visual>
-      <origin xyz="0 ${wheel_separation/2.0} ${wheel_radius}" rpy="0 1.5708 0"/>
+      <origin xyz="0 ${wheel_sep/2} ${wheel_radius}" rpy="0 1.5708 0"/>
       <geometry>
         <cylinder radius="${wheel_radius}" length="${wheel_width}"/>
       </geometry>
-      <material name="dark_grey">
-        <color rgba="0.2 0.2 0.2 1.0"/>
-      </material>
     </visual>
     <collision>
-      <origin xyz="0 ${wheel_separation/2.0} ${wheel_radius}" rpy="0 1.5708 0"/>
+      <origin xyz="0 ${wheel_sep/2} ${wheel_radius}"/>
       <geometry>
         <cylinder radius="${wheel_radius}" length="${wheel_width}"/>
       </geometry>
     </collision>
-    <xacro:inertial_box mass="0.5"
+    <xacro:inertial_box m="2.0"
                         x="${wheel_width}"
-                        y="${wheel_radius*2.0}"
-                        z="${wheel_radius*2.0}"/>
+                        y="${wheel_radius*2}"
+                        z="${wheel_radius*2}"/>
   </link>
   <joint name="left_wheel_joint" type="continuous">
     <parent link="base_link"/>
-    <child link="left_wheel_link"/>
-    <origin xyz="0 ${wheel_separation/2.0} ${wheel_radius}" rpy="0 0 0"/>
+    <child link="left_wheel"/>
+    <origin xyz="0 ${wheel_sep/2} ${wheel_radius}"/>
     <axis xyz="0 1 0"/>
   </joint>
-  <link name="right_wheel_link">
+  <link name="right_wheel">
     <visual>
-      <origin xyz="0 ${-wheel_separation/2.0} ${wheel_radius}" rpy="0 1.5708 0"/>
+      <origin xyz="0 ${-wheel_sep/2} ${wheel_radius}" rpy="0 1.5708 0"/>
       <geometry>
         <cylinder radius="${wheel_radius}" length="${wheel_width}"/>
       </geometry>
-      <material name="dark_grey"/>
     </visual>
     <collision>
-      <origin xyz="0 ${-wheel_separation/2.0} ${wheel_radius}" rpy="0 1.5708 0"/>
+      <origin xyz="0 ${-wheel_sep/2} ${wheel_radius}"/>
       <geometry>
         <cylinder radius="${wheel_radius}" length="${wheel_width}"/>
       </geometry>
     </collision>
-    <xacro:inertial_box mass="0.5"
+    <xacro:inertial_box m="2.0"
                         x="${wheel_width}"
-                        y="${wheel_radius*2.0}"
-                        z="${wheel_radius*2.0}"/>
+                        y="${wheel_radius*2}"
+                        z="${wheel_radius*2}"/>
   </link>
   <joint name="right_wheel_joint" type="continuous">
     <parent link="base_link"/>
-    <child link="right_wheel_link"/>
-    <origin xyz="0 ${-wheel_separation/2.0} ${wheel_radius}" rpy="0 0 0"/>
+    <child link="right_wheel"/>
+    <origin xyz="0 ${-wheel_sep/2} ${wheel_radius}"/>
     <axis xyz="0 1 0"/>
   </joint>
-  <!-- Caster -->
-  <link name="caster_wheel">
+  <!-- ================= FIXED FLAPS (GUIDES) ================= -->
+  <link name="left_flap">
     <visual>
-      <origin xyz="-${base_length/2.0 - 0.05} 0 ${wheel_radius/2.0}" rpy="0 0 0"/>
+      <origin xyz="0.30 0.30 0.20" rpy="0 0 -0.5"/>
       <geometry>
-        <sphere radius="${wheel_radius/2.0}"/>
+        <box size="0.60 0.05 0.35"/>
       </geometry>
-      <material name="dark_grey"/>
     </visual>
     <collision>
-      <origin xyz="-${base_length/2.0 - 0.05} 0 ${wheel_radius/2.0}" rpy="0 0 0"/>
+      <origin xyz="0.30 0.30 0.20" rpy="0 0 -0.5"/>
       <geometry>
-        <sphere radius="${wheel_radius/2.0}"/>
+        <box size="0.60 0.05 0.35"/>
       </geometry>
     </collision>
-    <xacro:inertial_box mass="0.2"
-                        x="${wheel_radius}"
-                        y="${wheel_radius}"
-                        z="${wheel_radius}"/>
+    <xacro:inertial_box m="4.0" x="0.6" y="0.05" z="0.35"/>
   </link>
-  <joint name="caster_joint" type="fixed">
+  <joint name="left_flap_joint" type="fixed">
     <parent link="base_link"/>
-    <child link="caster_wheel"/>
-    <origin xyz="-${base_length/2.0 - 0.05} 0 0" rpy="0 0 0"/>
+    <child link="left_flap"/>
+    <origin xyz="0 0 0"/>
   </joint>
-  <!-- Simple lidar puck -->
+  <link name="right_flap">
+    <visual>
+      <origin xyz="0.30 -0.30 0.20" rpy="0 0 0.5"/>
+      <geometry>
+        <box size="0.60 0.05 0.35"/>
+      </geometry>
+    </visual>
+    <collision>
+      <origin xyz="0.30 -0.30 0.20" rpy="0 0 0.5"/>
+      <geometry>
+        <box size="0.60 0.05 0.35"/>
+      </geometry>
+    </collision>
+    <xacro:inertial_box m="4.0" x="0.6" y="0.05" z="0.35"/>
+  </link>
+  <joint name="right_flap_joint" type="fixed">
+    <parent link="base_link"/>
+    <child link="right_flap"/>
+    <origin xyz="0 0 0"/>
+  </joint>
+  <!-- ================= LIDAR SENSOR ================= -->
   <link name="lidar_link">
     <visual>
-      <origin xyz="0 0 ${base_height + 0.05}" rpy="0 0 0"/>
+      <origin xyz="0.10 0 ${base_height + 0.15}"/>
       <geometry>
-        <cylinder radius="0.05" length="0.02"/>
+        <cylinder radius="0.06" length="0.08"/>
       </geometry>
-      <material name="lidar_body">
-        <color rgba="0.1 0.1 0.1 1.0"/>
-      </material>
     </visual>
     <collision>
-      <origin xyz="0 0 ${base_height + 0.05}" rpy="0 0 0"/>
+      <origin xyz="0.10 0 ${base_height + 0.15}"/>
       <geometry>
-        <cylinder radius="0.05" length="0.02"/>
+        <cylinder radius="0.06" length="0.08"/>
       </geometry>
     </collision>
-    <inertial>
-      <mass value="0.3"/>
-      <origin xyz="0 0 0" rpy="0 0 0"/>
-      <inertia ixx="0.0001" ixy="0.0" ixz="0.0"
-               iyy="0.0001" iyz="0.0" izz="0.0001"/>
-    </inertial>
+    <xacro:inertial_box m="0.3" x="0.08" y="0.08" z="0.08"/>
   </link>
   <joint name="lidar_joint" type="fixed">
     <parent link="base_link"/>
     <child link="lidar_link"/>
-    <origin xyz="0 0 0" rpy="0 0 0"/>
+    <origin xyz="0 0 0"/>
   </joint>
+  <!-- ================= DIFF DRIVE ================= -->
+  <gazebo>
+    <plugin filename="gz-sim-diff-drive-system"
+            name="gz::sim::systems::DiffDrive">
+      <left_joint>left_wheel_joint</left_joint>
+      <right_joint>right_wheel_joint</right_joint>
+      <wheel_separation>${wheel_sep}</wheel_separation>
+      <wheel_radius>${wheel_radius}</wheel_radius>
+      <topic>cmd_vel</topic>
+      <odom_topic>odom</odom_topic>
+      <frame_id>odom</frame_id>
+      <child_frame_id>base_link</child_frame_id>
+    </plugin>
+  </gazebo>
 </robot>
